Commit message: Fix ArUco detector startup and follow workflow

File: robot2/robot.urdf.xacro (robot description, xacro)
@@ -66,7 +66,5 @@
     <collision name="aruco_marker_collision">
       <geometry>
-        <box>
-          <size>0.01 0.4 0.4</size>
-        </box>
+        <box size="0.01 0.4 0.4"/>
       </geometry>
     </collision>
